File: ECAD/PowerChargeUSBHub/PowerChargeUSBHub.kicad_sch (KiCad schematic)
At the start: 0 parts

Commit message: WIP - first components
Parts:
- added D1: LED_Small, LED_THT:LED_D5.0mm_Horizontal_O1.27mm_Z3.0mm, symbol Device:LED_Small
- added D2, D3, D4: 1N5817, Diode_THT:D_DO-41_SOD81_P10.16mm_Horizontal, symbol Diode:1N5817
- added H1, H2: M3, MountingHole:MountingHole_3.2mm_M3_Pad_Via, symbol Mechanical:MountingHole_Pad
- added J1, J2, J3: USB_A, Connector_USB:USB_A_Molex_67643_Horizontal, symbol Connector:USB_A
- added JP1, JP2, JP3: SolderJumper_2_Open, Jumper:SolderJumper-2_P1.3mm_Open_Pad1.0x1.5mm, symbol Jumper:SolderJumper_2_Open
- added R1: R_Small, Resistor_SMD:R_1206_3216Metric_Pad1.30x1.75mm_HandSolder, symbol Device:R_Small
Connections:
- new net: D3.1 (K), J1.1 (VBUS), JP2.1 (A)
- new net: D1.2 (A), R1.2
- new net: D2.1 (K), J3.1 (VBUS), JP1.1 (A)
- new net: D4.1 (K), J2.1 (VBUS), JP3.1 (A)
- new net +5V: D2.2 (A), D3.2 (A), D4.2 (A), JP1.2 (B), JP2.2 (B), JP3.2 (B), R1.1
- new net GND: D1.1 (K), H1.1, H2.1, J1.4 (GND), J1.5 (Shield), J2.4 (GND), J2.5 (Shield), J3.4 (GND), J3.5 (Shield)
- no-connect marks 0 -> 6

Commit message: Add usbn C and polyfuse
Parts:
- added F1: Polyfuse_Small, PCM_Fuse_US_AKL:Fuse_Littelfuse-LVR200, symbol Device:Polyfuse_Small
- added J4: USB_C_Receptacle_PowerOnly_6P, Connector_USB:USB_C_Receptacle_GCT_USB4125-xx-x_6P_TopMnt_Horizontal, symbol Connector:USB_C_Receptacle_PowerOnly_6P
Connections:
- net +5V: now also F1.2
- net GND: now also J4.A12 (GND), J4.B12 (GND), J4.S1 (SHIELD)
- new net: F1.1, J4.A9 (VBUS), J4.B9 (VBUS)
- no-connect marks 6 -> 8
Changed lines of the file:
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@@
   (no_connect (at 128.27 58.42))
   (no_connect (at 95.25 58.42))
+  (no_connect (at 172.72 68.58))
   (no_connect (at 111.76 60.96))
   (no_connect (at 128.27 60.96))
+  (no_connect (at 172.72 71.12))
   (no_connect (at 111.76 58.42))
   (wire (pts (xy 95.25 44.45) (xy 99.06 44.45))
@@
     (stroke (width 0) (type default))
   )
+  (wire (pts (xy 184.15 49.53) (xy 184.15 55.88))
+    (stroke (width 0) (type default))
+  )
+  (wire (pts (xy 184.15 55.88) (xy 177.8 55.88))
+    (stroke (width 0) (type default))
+  )
   (wire (pts (xy 111.76 44.45) (xy 111.76 53.34))
     (stroke (width 0) (type default))
@@
         (path "/b12a6e25-97fb-4aba-bc96-af8db389bb9a"
           (reference "D3") (unit 1)
+        )
+      )
+    )
+  )
+  (symbol (lib_id "Device:Polyfuse_Small") (at 175.26 55.88 90) (unit 1)
+    (in_bom yes) (on_board yes) (dnp no) (fields_autoplaced)
+    (property "Reference" "F1" (at 175.26 49.53 90)
+      (effects (font (size 1.27 1.27)))
+    )
+    (property "Value" "Polyfuse_Small" (at 175.26 52.07 90)
+      (effects (font (size 1.27 1.27)))
+    )
+    (property "Footprint" "PCM_Fuse_US_AKL:Fuse_Littelfuse-LVR200" (at 180.34 54.61 0)
+      (effects (font (size 1.27 1.27)) (justify left) hide)
+    )
+    (property "Datasheet" "~" (at 175.26 55.88 0)
+      (effects (font (size 1.27 1.27)) hide)
+    )
+    (pin "1")
+    (pin "2")
+    (instances
+      (project "PowerChargeUSBHub"
+        (path "/b12a6e25-97fb-4aba-bc96-af8db389bb9a"
+          (reference "F1") (unit 1)
+        )
+      )
+    )
+  )
+  (symbol (lib_id "power:+5V") (at 184.15 49.53 0) (unit 1)
+    (in_bom yes) (on_board yes) (dnp no) (fields_autoplaced)
+    (property "Reference" "#PWR014" (at 184.15 53.34 0)
+      (effects (font (size 1.27 1.27)) hide)
+    )
+    (property "Value" "+5V" (at 184.15 44.45 0)
+      (effects (font (size 1.27 1.27)))
+    )
+    (property "Footprint" "" (at 184.15 49.53 0)
+      (effects (font (size 1.27 1.27)) hide)
+    )
+    (property "Datasheet" "" (at 184.15 49.53 0)
+      (effects (font (size 1.27 1.27)) hide)
+    )
+    (pin "1")
+    (instances
+      (project "PowerChargeUSBHub"
+        (path "/b12a6e25-97fb-4aba-bc96-af8db389bb9a"
+          (reference "#PWR014") (unit 1)
         )
       )
@@
     )
   )
+  (symbol (lib_id "Connector:USB_C_Receptacle_PowerOnly_6P") (at 157.48 63.5 0) (unit 1)
+    (in_bom yes) (on_board yes) (dnp no) (fields_autoplaced)
+    (property "Reference" "J4" (at 157.48 45.72 0)
+      (effects (font (size 1.27 1.27)))
+    )
+    (property "Value" "USB_C_Receptacle_PowerOnly_6P" (at 157.48 48.26 0)
+      (effects (font (size 1.27 1.27)))
+    )
+    (property "Footprint" "Connector_USB:USB_C_Receptacle_GCT_USB4125-xx-x_6P_TopMnt_Horizontal" (at 161.29 60.96 0)
+      (effects (font (size 1.27 1.27)) hide)
+    )
+    (property "Datasheet" "https://www.usb.org/sites/default/files/documents/usb_type-c.zip" (at 157.48 63.5 0)
+      (effects (font (size 1.27 1.27)) hide)
+    )
+    (pin "B12")
+    (pin "B9")
+    (pin "S1")
+    (pin "A12")
+    (pin "B5")
+    (pin "A5")
+    (pin "A9")
+    (instances
+      (project "PowerChargeUSBHub"
+        (path "/b12a6e25-97fb-4aba-bc96-af8db389bb9a"
+          (reference "J4") (unit 1)
+        )
+      )
+    )
+  )
+  (symbol (lib_id "power:GND") (at 149.86 81.28 0) (unit 1)
+    (in_bom yes) (on_board yes) (dnp no) (fields_autoplaced)
+    (property "Reference" "#PWR016" (at 149.86 87.63 0)
+      (effects (font (size 1.27 1.27)) hide)
+    )
+    (property "Value" "GND" (at 149.86 86.36 0)
+      (effects (font (size 1.27 1.27)))
+    )
+    (property "Footprint" "" (at 149.86 81.28 0)
+      (effects (font (size 1.27 1.27)) hide)
+    )
+    (property "Datasheet" "" (at 149.86 81.28 0)
+      (effects (font (size 1.27 1.27)) hide)
+    )
+    (pin "1")
+    (instances
+      (project "PowerChargeUSBHub"
+        (path "/b12a6e25-97fb-4aba-bc96-af8db389bb9a"
+          (reference "#PWR016") (unit 1)
+        )
+      )
+    )
+  )
   (symbol (lib_id "Diode:1N5817") (at 128.27 40.64 90) (unit 1)
     (in_bom yes) (on_board yes) (dnp no) (fields_autoplaced)
@@
         )
       )
+    )
+  )
+  (symbol (lib_id "power:GND") (at 157.48 81.28 0) (unit 1)
+    (in_bom yes) (on_board yes) (dnp no) (fields_autoplaced)
+    (property "Reference" "#PWR015" (at 157.48 87.63 0)
+      (effects (font (size 1.27 1.27)) hide)
+    )
+    (property "Value" "GND" (at 157.48 86.36 0)
+      (effects (font (size 1.27 1.27)))
+    )
+    (property "Footprint" "" (at 157.48 81.28 0)
+      (effects (font (size 1.27 1.27)) hide)
+    )
+    (property "Datasheet" "" (at 157.48 81.28 0)
+      (effects (font (size 1.27 1.27)) hide)
+    )
+    (pin "1")
+    (instances
+      (project "PowerChargeUSBHub"
+        (path "/b12a6e25-97fb-4aba-bc96-af8db389bb9a"
+          (reference "#PWR015") (unit 1)
+        )
+      )

Commit message: Create Dock
Parts:
- added H3, H4: M3, MountingHole:MountingHole_3.2mm_M3_Pad_Via, symbol Mechanical:MountingHole_Pad
Connections:
- net GND: now also H3.1, H4.1
- net at D3.1 (K), JP2.1 (A): now also J2.1 (VBUS); no longer J1.1 (VBUS)
- net at D4.1 (K), JP3.1 (A): now also J1.1 (VBUS); no longer J2.1 (VBUS)
Changed lines of the file:
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@@
+    )
+  )
+  (symbol (lib_id "power:GND") (at 49.53 66.04 0) (unit 1)
+    (in_bom yes) (on_board yes) (dnp no) (fields_autoplaced)
+    (property "Reference" "#PWR017" (at 49.53 72.39 0)
+      (effects (font (size 1.27 1.27)) hide)
+    )
+    (property "Value" "GND" (at 49.53 71.12 0)
+      (effects (font (size 1.27 1.27)))
+    )
+    (property "Footprint" "" (at 49.53 66.04 0)
+      (effects (font (size 1.27 1.27)) hide)
+    )
+    (property "Datasheet" "" (at 49.53 66.04 0)
+      (effects (font (size 1.27 1.27)) hide)
+    )
+    (pin "1")
+    (instances
+      (project "PowerChargeUSBHub"
+        (path "/b12a6e25-97fb-4aba-bc96-af8db389bb9a"
+          (reference "#PWR017") (unit 1)
+        )
+      )
     )
   )
@@
         (path "/b12a6e25-97fb-4aba-bc96-af8db389bb9a"
           (reference "F1") (unit 1)
+        )
+      )
+    )
+  )
+  (symbol (lib_id "Connector:USB_A") (at 104.14 58.42 0) (unit 1)
+    (in_bom yes) (on_board yes) (dnp no) (fields_autoplaced)
+    (property "Reference" "J1" (at 104.14 45.72 0)
+      (effects (font (size 1.27 1.27)))
+    )
+    (property "Value" "USB_A" (at 104.14 48.26 0)
+      (effects (font (size 1.27 1.27)))
+    )
+    (property "Footprint" "Connector_USB:USB_A_Molex_67643_Horizontal" (at 107.95 59.69 0)
+      (effects (font (size 1.27 1.27)) hide)
+    )
+    (property "Datasheet" " ~" (at 107.95 59.69 0)
+      (effects (font (size 1.27 1.27)) hide)
+    )
+    (pin "1")
+    (pin "2")
+    (pin "3")
+    (pin "4")
+    (pin "5")
+    (instances
+      (project "PowerChargeUSBHub"
+        (path "/b12a6e25-97fb-4aba-bc96-af8db389bb9a"
+          (reference "J1") (unit 1)
         )
       )
@@
       (effects (font (size 1.27 1.27)) hide)
     )
-    (pin "2")
-    (pin "1")
+    (pin "1")
+    (pin "2")
     (instances
       (project "PowerChargeUSBHub"
@@
     )
   )
+  (symbol (lib_id "power:GND") (at 57.15 66.04 0) (unit 1)
+    (in_bom yes) (on_board yes) (dnp no) (fields_autoplaced)
+    (property "Reference" "#PWR018" (at 57.15 72.39 0)
+      (effects (font (size 1.27 1.27)) hide)
+    )
+    (property "Value" "GND" (at 57.15 71.12 0)
+      (effects (font (size 1.27 1.27)))
+    )
+    (property "Footprint" "" (at 57.15 66.04 0)
+      (effects (font (size 1.27 1.27)) hide)
+    )
+    (property "Datasheet" "" (at 57.15 66.04 0)
+      (effects (font (size 1.27 1.27)) hide)
+    )
+    (pin "1")
+    (instances
+      (project "PowerChargeUSBHub"
+        (path "/b12a6e25-97fb-4aba-bc96-af8db389bb9a"
+          (reference "#PWR018") (unit 1)
+        )
+      )
+    )
+  )
   (symbol (lib_id "Connector:USB_C_Receptacle_PowerOnly_6P") (at 157.48 63.5 0) (unit 1)
     (in_bom yes) (on_board yes) (dnp no) (fields_autoplaced)
@@
       (effects (font (size 1.27 1.27)) hide)
     )
+    (pin "A12")
+    (pin "A5")
+    (pin "A9")
     (pin "B12")
+    (pin "B5")
     (pin "B9")
     (pin "S1")
-    (pin "A12")
-    (pin "B5")
-    (pin "A5")
-    (pin "A9")
     (instances
       (project "PowerChargeUSBHub"
@@
         (path "/b12a6e25-97fb-4aba-bc96-af8db389bb9a"
           (reference "D2") (unit 1)
-        )
-      )
-    )
-  )
-  (symbol (lib_id "Connector:USB_A") (at 87.63 58.42 0) (unit 1)
-    (in_bom yes) (on_board yes) (dnp no) (fields_autoplaced)
-    (property "Reference" "J1" (at 87.63 45.72 0)
-      (effects (font (size 1.27 1.27)))
-    )
-    (property "Value" "USB_A" (at 87.63 48.26 0)
-      (effects (font (size 1.27 1.27)))
-    )
-    (property "Footprint" "Connector_USB:USB_A_Molex_67643_Horizontal" (at 91.44 59.69 0)
-      (effects (font (size 1.27 1.27)) hide)
-    )
-    (property "Datasheet" " ~" (at 91.44 59.69 0)
-      (effects (font (size 1.27 1.27)) hide)
-    )
-    (pin "1")
-    (pin "2")
-    (pin "4")
-    (pin "3")
-    (pin "5")
-    (instances
-      (project "PowerChargeUSBHub"
-        (path "/b12a6e25-97fb-4aba-bc96-af8db389bb9a"
-          (reference "J1") (unit 1)
         )
       )
@@
       (effects (font (size 1.27 1.27)) hide)
     )
-    (pin "2")
-    (pin "1")
+    (pin "1")
+    (pin "2")
     (instances
       (project "PowerChargeUSBHub"
@@
     (pin "1")
     (pin "2")
+    (pin "3")
     (pin "4")
-    (pin "3")
     (pin "5")
     (instances
@@
       (effects (font (size 1.27 1.27)) hide)
     )
-    (pin "2")
-    (pin "1")
+    (pin "1")
+    (pin "2")
     (instances
       (project "PowerChargeUSBHub"
@@
     )
   )
+  (symbol (lib_id "Connector:USB_A") (at 87.63 58.42 0) (unit 1)
+    (in_bom yes) (on_board yes) (dnp no) (fields_autoplaced)
+    (property "Reference" "J2" (at 87.63 45.72 0)
+      (effects (font (size 1.27 1.27)))
+    )
+    (property "Value" "USB_A" (at 87.63 48.26 0)
+      (effects (font (size 1.27 1.27)))
+    )
+    (property "Footprint" "Connector_USB:USB_A_Molex_67643_Horizontal" (at 91.44 59.69 0)
+      (effects (font (size 1.27 1.27)) hide)
+    )
+    (property "Datasheet" " ~" (at 91.44 59.69 0)
+      (effects (font (size 1.27 1.27)) hide)
+    )
+    (pin "1")
+    (pin "2")
+    (pin "3")
+    (pin "4")
+    (pin "5")
+    (instances
+      (project "PowerChargeUSBHub"
+        (path "/b12a6e25-97fb-4aba-bc96-af8db389bb9a"
+          (reference "J2") (unit 1)
+        )
+      )
+    )
+  )
   (symbol (lib_id "power:+5V") (at 111.76 36.83 0) (unit 1)
     (in_bom yes) (on_board yes) (dnp no) (fields_autoplaced)
@@
     )
   )
+  (symbol (lib_id "Mechanical:MountingHole_Pad") (at 49.53 63.5 0) (unit 1)
+    (in_bom yes) (on_board yes) (dnp no) (fields_autoplaced)
+    (property "Reference" "H3" (at 52.07 60.96 0)
+      (effects (font (size 1.27 1.27)) (justify left))
+    )
+    (property "Value" "M3" (at 52.07 63.5 0)
+      (effects (font (size 1.27 1.27)) (justify left))
+    )
+    (property "Footprint" "MountingHole:MountingHole_3.2mm_M3_Pad_Via" (at 49.53 63.5 0)
+      (effects (font (size 1.27 1.27)) hide)
+    )
+    (property "Datasheet" "~" (at 49.53 63.5 0)
+      (effects (font (size 1.27 1.27)) hide)
+    )
+    (pin "1")
+    (instances
+      (project "PowerChargeUSBHub"
+        (path "/b12a6e25-97fb-4aba-bc96-af8db389bb9a"
+          (reference "H3") (unit 1)
+        )
+      )
+    )
+  )
   (symbol (lib_id "power:+5V") (at 128.27 36.83 0) (unit 1)
     (in_bom yes) (on_board yes) (dnp no) (fields_autoplaced)
@@
     )
   )
-  (symbol (lib_id "Connector:USB_A") (at 104.14 58.42 0) (unit 1)
-    (in_bom yes) (on_board yes) (dnp no) (fields_autoplaced)
-    (property "Reference" "J2" (at 104.14 45.72 0)
-      (effects (font (size 1.27 1.27)))
-    )
-    (property "Value" "USB_A" (at 104.14 48.26 0)
-      (effects (font (size 1.27 1.27)))
-    )
-    (property "Footprint" "Connector_USB:USB_A_Molex_67643_Horizontal" (at 107.95 59.69 0)
-      (effects (font (size 1.27 1.27)) hide)
-    )
-    (property "Datasheet" " ~" (at 107.95 59.69 0)
-      (effects (font (size 1.27 1.27)) hide)
-    )
-    (pin "1")
-    (pin "2")
-    (pin "4")
-    (pin "3")
-    (pin "5")
-    (instances
-      (project "PowerChargeUSBHub"
-        (path "/b12a6e25-97fb-4aba-bc96-af8db389bb9a"
-          (reference "J2") (unit 1)
-        )
-      )
-    )
-  )
   (symbol (lib_id "Diode:1N5817") (at 111.76 40.64 90) (unit 1)
     (in_bom yes) (on_board yes) (dnp no) (fields_autoplaced)
@@
         )
       )
+    )
+  )
+  (symbol (lib_id "Mechanical:MountingHole_Pad") (at 57.15 63.5 0) (unit 1)
+    (in_bom yes) (on_board yes) (dnp no) (fields_autoplaced)
+    (property "Reference" "H4" (at 59.69 60.96 0)
+      (effects (font (size 1.27 1.27)) (justify left))
+    )
+    (property "Value" "M3" (at 59.69 63.5 0)
+      (effects (font (size 1.27 1.27)) (justify left))
+    )
+    (property "Footprint" "MountingHole:MountingHole_3.2mm_M3_Pad_Via" (at 57.15 63.5 0)
+      (effects (font (size 1.27 1.27)) hide)
+    )
+    (property "Datasheet" "~" (at 57.15 63.5 0)
+      (effects (font (size 1.27 1.27)) hide)
+    )
+    (pin "1")
+    (instances
+      (project "PowerChargeUSBHub"
+        (path "/b12a6e25-97fb-4aba-bc96-af8db389bb9a"
+          (reference "H4") (unit 1)
+        )
+      )
